File: schematics/src/ioboard/ioboard.sch (EAGLE design)
At the start: 18 parts

Commit message: fixed headers
Parts:
- removed +12V, -12V, GND, JP2: (no value), pinhead:PINHD-1X3
- added JP1, JP3: (no value), pinhead:PINHD-2X3
Connections:
- net +12V: now also JP1.2, JP1.4, JP1.6; no longer +12V.1, +12V.2, +12V.3
- net -12V: now also JP3.1, JP3.3, JP3.5; no longer -12V.1, -12V.2, -12V.3
- net N$6: now also JP1.1, JP1.3, JP1.5; no longer JP2.1, JP2.2, JP2.3
- net N$9: now also JP3.2, JP3.4, JP3.6; no longer GND.1, GND.2, GND.3
Changed lines of the file:
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@@
 <part name="P-1" library="supply1" deviceset="-12V" device=""/>
 <part name="GND2" library="supply1" deviceset="GND" device=""/>
-<part name="+12V" library="pinhead" library_urn="urn:adsk.eagle:library:325" deviceset="PINHD-1X3" device="" package3d_urn="urn:adsk.eagle:package:22458/2"/>
-<part name="JP2" library="pinhead" library_urn="urn:adsk.eagle:library:325" deviceset="PINHD-1X3" device="" package3d_urn="urn:adsk.eagle:package:22458/2"/>
-<part name="GND" library="pinhead" library_urn="urn:adsk.eagle:library:325" deviceset="PINHD-1X3" device="" package3d_urn="urn:adsk.eagle:package:22458/2"/>
-<part name="-12V" library="pinhead" library_urn="urn:adsk.eagle:library:325" deviceset="PINHD-1X3" device="" package3d_urn="urn:adsk.eagle:package:22458/2"/>
 <part name="JP5" library="pinhead" library_urn="urn:adsk.eagle:library:325" deviceset="PINHD-1X4" device="" package3d_urn="urn:adsk.eagle:package:22407/2"/>
 <part name="P+2" library="supply1" deviceset="+12V" device=""/>
@@
 <part name="JP9" library="pinhead" library_urn="urn:adsk.eagle:library:325" deviceset="PINHD-1X2" device="" package3d_urn="urn:adsk.eagle:package:22435/2"/>
 <part name="GND9" library="supply1" deviceset="GND" device=""/>
+<part name="JP1" library="pinhead" library_urn="urn:adsk.eagle:library:325" deviceset="PINHD-2X3" device="" package3d_urn="urn:adsk.eagle:package:22462/2"/>
+<part name="JP3" library="pinhead" library_urn="urn:adsk.eagle:library:325" deviceset="PINHD-2X3" device="" package3d_urn="urn:adsk.eagle:package:22462/2"/>
 </parts>
 <sheets>
@@
 <attribute name="VALUE" x="81.28" y="63.5" size="1.778" layer="96"/>
 </instance>
-<instance part="+12V" gate="A" x="223.52" y="137.16" smashed="yes">
-<attribute name="NAME" x="217.17" y="142.875" size="1.778" layer="95"/>
-<attribute name="VALUE" x="217.17" y="129.54" size="1.778" layer="96"/>
-</instance>
-<instance part="JP2" gate="A" x="223.52" y="114.3" smashed="yes">
-<attribute name="NAME" x="217.17" y="120.015" size="1.778" layer="95"/>
-<attribute name="VALUE" x="217.17" y="106.68" size="1.778" layer="96"/>
-</instance>
-<instance part="GND" gate="A" x="223.52" y="91.44" smashed="yes">
-<attribute name="NAME" x="217.17" y="97.155" size="1.778" layer="95"/>
-<attribute name="VALUE" x="217.17" y="83.82" size="1.778" layer="96"/>
-</instance>
-<instance part="-12V" gate="A" x="223.52" y="68.58" smashed="yes">
-<attribute name="NAME" x="217.17" y="74.295" size="1.778" layer="95"/>
-<attribute name="VALUE" x="217.17" y="60.96" size="1.778" layer="96"/>
-</instance>
 <instance part="JP5" gate="A" x="30.48" y="147.32" smashed="yes" rot="R180">
 <attribute name="NAME" x="36.83" y="139.065" size="1.778" layer="95" rot="R180"/>
 <attribute name="VALUE" x="36.83" y="154.94" size="1.778" layer="96" rot="R180"/>
 </instance>
-<instance part="P+2" gate="1" x="213.36" y="147.32" smashed="yes">
-<attribute name="VALUE" x="210.82" y="142.24" size="1.778" layer="96" rot="R90"/>
-</instance>
-<instance part="P-2" gate="1" x="213.36" y="58.42" smashed="yes">
-<attribute name="VALUE" x="210.82" y="55.88" size="1.778" layer="96" rot="R90"/>
+<instance part="P+2" gate="1" x="236.22" y="124.46" smashed="yes" rot="MR0">
+<attribute name="VALUE" x="238.76" y="119.38" size="1.778" layer="96" rot="MR90"/>
+</instance>
+<instance part="P-2" gate="1" x="236.22" y="78.74" smashed="yes">
+<attribute name="VALUE" x="233.68" y="76.2" size="1.778" layer="96" rot="R90"/>
 </instance>
 <instance part="JP6" gate="G$1" x="203.2" y="101.6" smashed="yes" rot="R270">
@@
 <instance part="GND9" gate="1" x="170.18" y="88.9" smashed="yes">
 <attribute name="VALUE" x="167.64" y="86.36" size="1.778" layer="96"/>
+</instance>
+<instance part="JP1" gate="A" x="223.52" y="114.3" smashed="yes">
+<attribute name="NAME" x="217.17" y="120.015" size="1.778" layer="95"/>
+<attribute name="VALUE" x="217.17" y="106.68" size="1.778" layer="96"/>
+</instance>
+<instance part="JP3" gate="A" x="226.06" y="91.44" smashed="yes" rot="R180">
+<attribute name="NAME" x="232.41" y="85.725" size="1.778" layer="95" rot="R180"/>
+<attribute name="VALUE" x="232.41" y="99.06" size="1.778" layer="96" rot="R180"/>
 </instance>
 </instances>
@@
 </segment>
 <segment>
-<pinref part="+12V" gate="A" pin="3"/>
-<wire x1="220.98" y1="134.62" x2="213.36" y2="134.62" width="0.1524" layer="91"/>
-<pinref part="+12V" gate="A" pin="2"/>
-<wire x1="220.98" y1="137.16" x2="213.36" y2="137.16" width="0.1524" layer="91"/>
-<wire x1="213.36" y1="134.62" x2="213.36" y2="137.16" width="0.1524" layer="91"/>
-<pinref part="+12V" gate="A" pin="1"/>
-<wire x1="220.98" y1="139.7" x2="213.36" y2="139.7" width="0.1524" layer="91"/>
-<wire x1="213.36" y1="137.16" x2="213.36" y2="139.7" width="0.1524" layer="91"/>
-<junction x="213.36" y="137.16"/>
-<wire x1="213.36" y1="139.7" x2="213.36" y2="144.78" width="0.1524" layer="91"/>
-<junction x="213.36" y="139.7"/>
+<wire x1="228.6" y1="111.76" x2="236.22" y2="111.76" width="0.1524" layer="91"/>
+<wire x1="228.6" y1="114.3" x2="236.22" y2="114.3" width="0.1524" layer="91"/>
+<wire x1="236.22" y1="111.76" x2="236.22" y2="114.3" width="0.1524" layer="91"/>
+<wire x1="228.6" y1="116.84" x2="236.22" y2="116.84" width="0.1524" layer="91"/>
+<wire x1="236.22" y1="114.3" x2="236.22" y2="116.84" width="0.1524" layer="91"/>
+<junction x="236.22" y="114.3"/>
+<wire x1="236.22" y1="116.84" x2="236.22" y2="121.92" width="0.1524" layer="91"/>
+<junction x="236.22" y="116.84"/>
 <pinref part="P+2" gate="1" pin="+12V"/>
+<pinref part="JP1" gate="A" pin="2"/>
+<pinref part="JP1" gate="A" pin="4"/>
+<pinref part="JP1" gate="A" pin="6"/>
 </segment>
 </net>
@@
 </segment>
 <segment>
-<pinref part="-12V" gate="A" pin="1"/>
-<wire x1="220.98" y1="71.12" x2="213.36" y2="71.12" width="0.1524" layer="91"/>
-<pinref part="-12V" gate="A" pin="2"/>
-<wire x1="220.98" y1="68.58" x2="213.36" y2="68.58" width="0.1524" layer="91"/>
-<wire x1="213.36" y1="71.12" x2="213.36" y2="68.58" width="0.1524" layer="91"/>
-<pinref part="-12V" gate="A" pin="3"/>
-<wire x1="220.98" y1="66.04" x2="213.36" y2="66.04" width="0.1524" layer="91"/>
-<wire x1="213.36" y1="68.58" x2="213.36" y2="66.04" width="0.1524" layer="91"/>
-<junction x="213.36" y="68.58"/>
-<wire x1="213.36" y1="66.04" x2="213.36" y2="60.96" width="0.1524" layer="91"/>
-<junction x="213.36" y="66.04"/>
+<wire x1="228.6" y1="88.9" x2="236.22" y2="88.9" width="0.1524" layer="91"/>
+<wire x1="228.6" y1="91.44" x2="236.22" y2="91.44" width="0.1524" layer="91"/>
+<wire x1="228.6" y1="93.98" x2="236.22" y2="93.98" width="0.1524" layer="91"/>
+<wire x1="236.22" y1="93.98" x2="236.22" y2="88.9" width="0.1524" layer="91"/>
+<wire x1="236.22" y1="91.44" x2="236.22" y2="88.9" width="0.1524" layer="91"/>
+<junction x="236.22" y="91.44"/>
+<wire x1="236.22" y1="88.9" x2="236.22" y2="81.28" width="0.1524" layer="91"/>
 <pinref part="P-2" gate="1" pin="-12V"/>
+<pinref part="JP3" gate="A" pin="1"/>
+<pinref part="JP3" gate="A" pin="3"/>
+<pinref part="JP3" gate="A" pin="5"/>
+<junction x="236.22" y="88.9"/>
 </segment>
 </net>
@@
 <net name="N$6" class="0">
 <segment>
-<pinref part="JP2" gate="A" pin="1"/>
 <wire x1="220.98" y1="116.84" x2="213.36" y2="116.84" width="0.1524" layer="91"/>
-<pinref part="JP2" gate="A" pin="2"/>
 <wire x1="220.98" y1="114.3" x2="213.36" y2="114.3" width="0.1524" layer="91"/>
 <wire x1="213.36" y1="116.84" x2="213.36" y2="114.3" width="0.1524" layer="91"/>
-<pinref part="JP2" gate="A" pin="3"/>
 <wire x1="220.98" y1="111.76" x2="213.36" y2="111.76" width="0.1524" layer="91"/>
 <wire x1="213.36" y1="114.3" x2="213.36" y2="111.76" width="0.1524" layer="91"/>
@@
 <pinref part="JP6" gate="G$1" pin="1"/>
 <wire x1="205.74" y1="109.22" x2="205.74" y2="104.14" width="0.1524" layer="91"/>
+<pinref part="JP1" gate="A" pin="1"/>
+<pinref part="JP1" gate="A" pin="3"/>
+<pinref part="JP1" gate="A" pin="5"/>
 </segment>
 </net>
 <net name="N$9" class="0">
 <segment>
-<pinref part="GND" gate="A" pin="1"/>
 <wire x1="220.98" y1="93.98" x2="213.36" y2="93.98" width="0.1524" layer="91"/>
-<pinref part="GND" gate="A" pin="2"/>
 <wire x1="220.98" y1="91.44" x2="213.36" y2="91.44" width="0.1524" layer="91"/>
 <wire x1="213.36" y1="93.98" x2="213.36" y2="91.44" width="0.1524" layer="91"/>
-<pinref part="GND" gate="A" pin="3"/>
 <wire x1="220.98" y1="88.9" x2="213.36" y2="88.9" width="0.1524" layer="91"/>
 <wire x1="213.36" y1="91.44" x2="213.36" y2="88.9" width="0.1524" layer="91"/>
@@
 <pinref part="GND_JMP" gate="G$1" pin="1"/>
 <wire x1="205.74" y1="86.36" x2="205.74" y2="81.28" width="0.1524" layer="91"/>
-</segment>
-</net>
+<pinref part="JP3" gate="A" pin="2"/>
+<pinref part="JP3" gate="A" pin="4"/>
+<pinref part="JP3" gate="A" pin="6"/>
+</segment>
+</net>
